Commit message: made a sim bringup file

File: install/new_robot_description/share/new_robot_description/urdf/laser.xacro (robot description, xacro)
@@ -21,5 +21,5 @@
         <parent link="base_link"/>
         <child link="laser_sensor_link"/>
-        <origin xyz="0.0 0.0 0.2"/>
+        <origin xyz="0.0 0.0 0.21"/>
     </joint>
     <gazebo reference="laser_sensor_link">
