Commit message: added camera

File: install/new_robot_description/share/new_robot_description/urdf/camera.xacro (robot description, xacro)
@@ -1,44 +1,49 @@
 <?xml version="1.0"?>
-<robot xmlns:xacro="http://www.ros.org/wiki/xacro">
+<robot xmlns:xacro="http://www.ros.org/wiki/xacro" >
     <link name="camera_frame">
         <visual>
             <geometry>
-                <box size= "0.010 0.03 0.03"/>
+                <box size="0.010 0.03 0.03"/>
             </geometry>
             <material name="grey"/>
         </visual>
     </link>
-    <joint name="base_laser_joint" type="fixed">
+    <joint name="base_camera_joint" type="fixed">
         <parent link="base_link"/>
         <child link="camera_frame"/>
-        <origin xyz="0.1 0.0 0.21" rpy = "0 0 0"/>
+        <origin xyz="0.1 0.0 0.21" rpy="0 0 0"/>
     </joint>
+    <joint name="camera_optical_joint" type="fixed">
+        <parent link="camera_frame"/>
+        <child link="camera_link_optical"/>
+        <origin xyz="0 0 0" rpy="${-pi/2} 0 ${-pi/2}"/>
+    </joint>
+    <link name="camera_link_optical"></link>
     <gazebo reference="camera_frame">
-        <material>Gazebo/Yellow</material>
-        <sensor name="laser" type="ray">
-            <pose> 0 0 0 0 0 0 </pose>
+        <sensor name="camera" type="camera">
+            <pose>0 0 0 0 0 0</pose>
             <visualize>true</visualize>
-            <update_rate>10</update_rate>
-            <ray>
-                <scan>
-                    <horizontal>
-                        <samples>360</samples>
-                        <min_angle>-3.14</min_angle>
-                        <max_angle>3.14</max_angle>
-                    </horizontal>
-                </scan>
-                <range>
-                    <min>0.3</min>
-                    <max>12</max>
-                </range>
-            </ray>
-            <plugin name="laser_controller" filename="libgazebo_ros_ray_sensor.so">
+            <update_rate>30</update_rate>
+            <camera>
+                <horizontal_fov>1.089</horizontal_fov>
+                <image>
+                    <format>R8G8B8</format>
+                    <width>640</width>
+                    <height>480</height>
+                </image>
+                <clip>
+                    <near>0.05</near>
+                    <far>8.0</far>
+                </clip>
+            </camera>
+            <plugin name="camera_controller" filename="libgazebo_ros_camera.so">
                 <ros>
-                    <argument>~/out:=scan</argument>
+                    <namespace>/camera</namespace>
+                    <argument>~/image_raw:=image_raw</argument>
                 </ros>
-                <output_type>sensor_msgs/LaserScan</output_type>
-                <frame_name>laser_sensor_link</frame_name>
+                <camera_name>camera</camera_name>
+                <frame_name>camera_link_optical</frame_name>
             </plugin>
         </sensor>
     </gazebo>
-    </robot>
+</robot>

File: src/new_robot_description/urdf/camera.xacro (robot description, xacro)
@@ -14,4 +14,10 @@
         <origin xyz="0.1 0.0 0.21" rpy="0 0 0"/>
     </joint>
+    <joint name="camera_optical_joint" type="fixed">
+        <parent link="camera_frame"/>
+        <child link="camera_link_optical"/>
+        <origin xyz="0 0 0" rpy="${-pi/2} 0 ${-pi/2}"/>
+    </joint>
+    <link name="camera_link_optical"></link>
     <gazebo reference="camera_frame">
         <sensor name="camera" type="camera">
@@ -20,13 +26,13 @@
             <update_rate>30</update_rate>
             <camera>
-                <horizontal_fov>1.3962634</horizontal_fov>
+                <horizontal_fov>1.089</horizontal_fov>
                 <image>
+                    <format>R8G8B8</format>
                     <width>640</width>
                     <height>480</height>
-                    <format>R8G8B8</format>
                 </image>
                 <clip>
-                    <near>0.1</near>
-                    <far>100</far>
+                    <near>0.05</near>
+                    <far>8.0</far>
                 </clip>
             </camera>
@@ -37,5 +43,5 @@
                 </ros>
                 <camera_name>camera</camera_name>
-                <frame_name>camera_frame</frame_name>
+                <frame_name>camera_link_optical</frame_name>
             </plugin>
         </sensor>
